File: CRSpill.sch (EAGLE design)
At the start: 23 parts, among them IC1 7805DT, IC2 BLUE_PILL, IC3 NCV7351D1E, J3 MA04-1, SW1 SWITCH_TACTILETOP, U1 STM32F103C8, U7 XC6206, X1 8P8C-LED

Commit message: 5V12Vの配線を強化
Connections:
- removed net LED0: IC2.B0
- removed net LED1: IC2.B1
- net PB0: now also IC2.B0
- net PB1: now also IC2.B1
Changed lines of the file:
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@@
 <class number="0" name="default" width="0" drill="0">
+</class>
+<class number="1" name="12v" width="0.5" drill="0">
 </class>
 </classes>
@@
 </segment>
 </net>
-<net name="N$2" class="0">
+<net name="N$2" class="1">
 <segment>
 <pinref part="X1" gate="G$1" pin="4"/>
@@
 </segment>
 </net>
-<net name="N$3" class="0">
+<net name="N$3" class="1">
 <segment>
 <pinref part="F1" gate="G$1" pin="1"/>
@@
 </segment>
 </net>
-<net name="+5V" class="0">
+<net name="+5V" class="1">
 <segment>
 <pinref part="P+1" gate="1" pin="+5V"/>
@@
 </segment>
 </net>
-<net name="LED0" class="0">
-<segment>
-<pinref part="IC2" gate="G$1" pin="B0"/>
-<wire x1="25.4" y1="91.44" x2="20.32" y2="91.44" width="0.1524" layer="91"/>
-<label x="20.32" y="91.44" size="1.778" layer="95" rot="R180" xref="yes"/>
-</segment>
-</net>
-<net name="LED1" class="0">
-<segment>
-<pinref part="IC2" gate="G$1" pin="B1"/>
-<wire x1="25.4" y1="88.9" x2="20.32" y2="88.9" width="0.1524" layer="91"/>
-<label x="20.32" y="88.9" size="1.778" layer="95" rot="R180" xref="yes"/>
-</segment>
-</net>
 <net name="SWDIO" class="0">
 <segment>
@@
 <label x="299.72" y="71.12" size="1.778" layer="95" rot="R270" xref="yes"/>
 </segment>
+<segment>
+<pinref part="IC2" gate="G$1" pin="B0"/>
+<wire x1="25.4" y1="91.44" x2="20.32" y2="91.44" width="0.1524" layer="91"/>
+<label x="20.32" y="91.44" size="1.778" layer="95" rot="R180" xref="yes"/>
+</segment>
 </net>
 <net name="PB5" class="0">
@@
 <label x="302.26" y="71.12" size="1.778" layer="95" rot="R270" xref="yes"/>
 </segment>
-</net>
+<segment>
+<pinref part="IC2" gate="G$1" pin="B1"/>
+<wire x1="25.4" y1="88.9" x2="20.32" y2="88.9" width="0.1524" layer="91"/>
+<label x="20.32" y="88.9" size="1.778" layer="95" rot="R180" xref="yes"/>
+</segment>
+</net>
