File: CRSpill.sch (EAGLE design)
At the start: 23 parts, among them IC1 7805DT, IC2 BLUE_PILL, IC3 NCV7351D1E, J3 MA04-1, SW1 SWITCH_TACTILETOP, U1 STM32F103C8, U7 XC6206, X1 8P8C-LED

Commit message: boot0他
Parts:
- added BOOT0: (no value), jumper:SJ2W
Connections:
- net +3V3: now also BOOT0.1
- net BOOT0: now also BOOT0.2
- net GND: now also BOOT0.3
Changed lines of the file:
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@@
 <layer number="56" name="wert" color="7" fill="1" visible="no" active="no"/>
 <layer number="57" name="tCAD" color="7" fill="1" visible="no" active="no"/>
+<layer number="59" name="tCarbon" color="7" fill="1" visible="no" active="no"/>
+<layer number="60" name="bCarbon" color="7" fill="1" visible="no" active="no"/>
 <layer number="88" name="SimResults" color="9" fill="1" visible="yes" active="yes"/>
 <layer number="89" name="SimProbes" color="9" fill="1" visible="yes" active="yes"/>
@@
 <layer number="112" name="tSilk" color="7" fill="1" visible="yes" active="yes"/>
 <layer number="113" name="IDFDebug" color="4" fill="1" visible="yes" active="yes"/>
+<layer number="114" name="Badge_Outline" color="7" fill="1" visible="no" active="yes"/>
+<layer number="115" name="ReferenceISLANDS" color="7" fill="1" visible="no" active="yes"/>
 <layer number="116" name="Patch_BOT" color="9" fill="4" visible="yes" active="yes"/>
+<layer number="118" name="Rect_Pads" color="7" fill="1" visible="no" active="yes"/>
 <layer number="121" name="_tsilk" color="7" fill="1" visible="yes" active="yes"/>
 <layer number="122" name="_bsilk" color="7" fill="1" visible="yes" active="yes"/>
@@
 <layer number="127" name="_tValues" color="7" fill="1" visible="yes" active="yes"/>
 <layer number="128" name="_bValues" color="7" fill="1" visible="yes" active="yes"/>
+<layer number="129" name="Mask" color="7" fill="1" visible="yes" active="yes"/>
 <layer number="131" name="tAdjust" color="7" fill="1" visible="yes" active="yes"/>
 <layer number="132" name="bAdjust" color="7" fill="1" visible="yes" active="yes"/>
@@
 <layer number="230" name="230bmp" color="7" fill="1" visible="yes" active="yes"/>
 <layer number="231" name="231bmp" color="7" fill="1" visible="yes" active="yes"/>
+<layer number="232" name="Eagle3D_PG2" color="7" fill="1" visible="yes" active="yes"/>
+<layer number="233" name="Eagle3D_PG3" color="7" fill="1" visible="yes" active="yes"/>
 <layer number="248" name="Housing" color="7" fill="1" visible="yes" active="yes"/>
 <layer number="249" name="Edge" color="7" fill="1" visible="yes" active="yes"/>
@@
 <layer number="251" name="SMDround" color="12" fill="11" visible="no" active="no"/>
 <layer number="254" name="cooling" color="7" fill="1" visible="yes" active="yes"/>
+<layer number="255" name="routoute" color="7" fill="1" visible="yes" active="yes"/>
 </layers>
 <schematic xreflabel="%F%N/%S.%C%R" xrefpart="/%S.%C%R">
@@
 <part name="J3" library="con-headers" deviceset="MA04-1" device=""/>
 <part name="GND21" library="supply1" library_urn="urn:adsk.eagle:library:371" deviceset="GNDA" device=""/>
+<part name="GND40" library="supply1" library_urn="urn:adsk.eagle:library:371" deviceset="GNDA" device=""/>
+<part name="+3V6" library="supply1" library_urn="urn:adsk.eagle:library:371" deviceset="+3V3" device=""/>
+<part name="BOOT0" library="jumper" library_urn="urn:adsk.eagle:library:252" deviceset="SJ2W" device="" package3d_urn="urn:adsk.eagle:package:15474/1"/>
 </parts>
 <sheets>
@@
 </instance>
 <instance part="GND21" gate="1" x="223.52" y="71.12" smashed="yes"/>
+<instance part="GND40" gate="1" x="137.16" y="73.66" smashed="yes"/>
+<instance part="+3V6" gate="G$1" x="154.94" y="88.9" smashed="yes">
+<attribute name="VALUE" x="152.4" y="83.82" size="1.778" layer="96" rot="R90"/>
+</instance>
+<instance part="BOOT0" gate="G$1" x="144.78" y="78.74" smashed="yes" rot="R270">
+<attribute name="NAME" x="145.161" y="76.2" size="1.778" layer="95" rot="R270"/>
+<attribute name="VALUE" x="142.875" y="76.2" size="1.778" layer="96" rot="R270"/>
+</instance>
 </instances>
 <busses>
@@
 <pinref part="GND21" gate="1" pin="GNDA"/>
 <label x="220.98" y="68.58" size="1.778" layer="95"/>
+</segment>
+<segment>
+<pinref part="GND40" gate="1" pin="GNDA"/>
+<wire x1="137.16" y1="76.2" x2="137.16" y2="78.74" width="0.1524" layer="91"/>
+<pinref part="BOOT0" gate="G$1" pin="3"/>
+<wire x1="137.16" y1="78.74" x2="139.7" y2="78.74" width="0.1524" layer="91"/>
+<label x="137.16" y="78.74" size="1.778" layer="95" rot="R90" xref="yes"/>
 </segment>
 </net>
@@
 <pinref part="J3" gate="G$1" pin="1"/>
 </segment>
+<segment>
+<pinref part="+3V6" gate="G$1" pin="+3V3"/>
+<pinref part="BOOT0" gate="G$1" pin="1"/>
+<wire x1="149.86" y1="78.74" x2="154.94" y2="78.74" width="0.1524" layer="91"/>
+<wire x1="154.94" y1="78.74" x2="154.94" y2="86.36" width="0.1524" layer="91"/>
+</segment>
 </net>
 <net name="N$9" class="0">
@@
 <label x="297.18" y="160.02" size="1.778" layer="95" rot="R90" xref="yes"/>
 </segment>
+<segment>
+<wire x1="144.78" y1="91.44" x2="144.78" y2="83.82" width="0.1524" layer="91"/>
+<pinref part="BOOT0" gate="G$1" pin="2"/>
+<label x="144.78" y="91.44" size="1.778" layer="95" rot="R90" xref="yes"/>
+</segment>
 </net>
 <net name="PB2" class="0">
@@
 </sheet>
 </sheets>
+<errors>
+</errors>
 </schematic>
 </drawing>

Commit message: 電解コンデンサ1個表面実装用に変更
Parts:
- removed C17: 22u, rcl:CPOL-EUE2-5
- added C5: 1u, rcl:C-EUC0603
Connections:
- net +5V: now also C5.1; no longer C17.+
- net GND: now also C5.2; no longer C17.-
Changed lines of the file:
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@@
 <part name="GND31" library="supply1" library_urn="urn:adsk.eagle:library:371" deviceset="GNDIO" device=""/>
 <part name="GND11" library="supply1" library_urn="urn:adsk.eagle:library:371" deviceset="GNDIO" device=""/>
-<part name="C17" library="rcl" deviceset="CPOL-EU" device="E2-5" value="22u"/>
 <part name="C16" library="rcl" deviceset="C-EU" device="C0603" value="100n"/>
 <part name="C18" library="rcl" deviceset="C-EU" device="C0603" value="100n"/>
-<part name="GND44" library="supply1" library_urn="urn:adsk.eagle:library:371" deviceset="GNDIO" device=""/>
 <part name="GND45" library="supply1" library_urn="urn:adsk.eagle:library:371" deviceset="GNDIO" device=""/>
 <part name="GND46" library="supply1" library_urn="urn:adsk.eagle:library:371" deviceset="GNDIO" device=""/>
@@
 <part name="+3V6" library="supply1" library_urn="urn:adsk.eagle:library:371" deviceset="+3V3" device=""/>
 <part name="BOOT0" library="jumper" library_urn="urn:adsk.eagle:library:252" deviceset="SJ2W" device="" package3d_urn="urn:adsk.eagle:package:15474/1"/>
+<part name="C5" library="rcl" deviceset="C-EU" device="C0603" value="1u"/>
+<part name="GND12" library="supply1" library_urn="urn:adsk.eagle:library:371" deviceset="GNDIO" device=""/>
 </parts>
 <sheets>
@@
 <instance part="GND31" gate="G$1" x="208.28" y="104.14" smashed="yes"/>
 <instance part="GND11" gate="G$1" x="289.56" y="160.02" smashed="yes" rot="R180"/>
-<instance part="C17" gate="G$1" x="48.26" y="30.48" smashed="yes">
-<attribute name="NAME" x="49.403" y="30.9626" size="1.778" layer="95"/>
-<attribute name="VALUE" x="49.403" y="25.8826" size="1.778" layer="96"/>
-</instance>
 <instance part="C16" gate="G$1" x="58.42" y="30.48" smashed="yes">
 <attribute name="NAME" x="59.944" y="30.861" size="1.778" layer="95"/>
@@
 <attribute name="VALUE" x="100.584" y="25.781" size="1.778" layer="96"/>
 </instance>
-<instance part="GND44" gate="G$1" x="48.26" y="17.78" smashed="yes"/>
 <instance part="GND45" gate="G$1" x="58.42" y="17.78" smashed="yes"/>
 <instance part="GND46" gate="G$1" x="88.9" y="17.78" smashed="yes"/>
@@
 <attribute name="VALUE" x="142.875" y="76.2" size="1.778" layer="96" rot="R270"/>
 </instance>
+<instance part="C5" gate="G$1" x="48.26" y="30.48" smashed="yes">
+<attribute name="NAME" x="49.784" y="30.861" size="1.778" layer="95"/>
+<attribute name="VALUE" x="49.784" y="25.781" size="1.778" layer="96"/>
+</instance>
+<instance part="GND12" gate="G$1" x="48.26" y="17.78" smashed="yes"/>
 </instances>
 <busses>
@@
 </segment>
 <segment>
-<pinref part="C17" gate="G$1" pin="-"/>
-<wire x1="48.26" y1="25.4" x2="48.26" y2="20.32" width="0.1524" layer="91"/>
-<pinref part="GND44" gate="G$1" pin="GNDIO"/>
-<label x="48.26" y="17.78" size="1.778" layer="95" xref="yes"/>
-</segment>
-<segment>
 <pinref part="C16" gate="G$1" pin="2"/>
 <wire x1="58.42" y1="20.32" x2="58.42" y2="25.4" width="0.1524" layer="91"/>
@@
 <wire x1="137.16" y1="78.74" x2="139.7" y2="78.74" width="0.1524" layer="91"/>
 <label x="137.16" y="78.74" size="1.778" layer="95" rot="R90" xref="yes"/>
+</segment>
+<segment>
+<wire x1="48.26" y1="20.32" x2="48.26" y2="25.4" width="0.1524" layer="91"/>
+<pinref part="GND12" gate="G$1" pin="GNDIO"/>
+<label x="48.26" y="17.78" size="1.778" layer="95" xref="yes"/>
+<pinref part="C5" gate="G$1" pin="2"/>
 </segment>
 </net>
@@
 <wire x1="63.5" y1="38.1" x2="58.42" y2="38.1" width="0.1524" layer="91"/>
 <wire x1="48.26" y1="38.1" x2="58.42" y2="38.1" width="0.1524" layer="91"/>
-<pinref part="C17" gate="G$1" pin="+"/>
-<wire x1="48.26" y1="33.02" x2="48.26" y2="38.1" width="0.1524" layer="91"/>
 <pinref part="C16" gate="G$1" pin="1"/>
 <wire x1="58.42" y1="38.1" x2="58.42" y2="33.02" width="0.1524" layer="91"/>
@@
 <pinref part="P+17" gate="1" pin="+5V"/>
 <wire x1="48.26" y1="48.26" x2="48.26" y2="38.1" width="0.1524" layer="91"/>
+<pinref part="U7" gate="G$1" pin="VIN"/>
+<pinref part="C5" gate="G$1" pin="1"/>
+<wire x1="48.26" y1="33.02" x2="48.26" y2="38.1" width="0.1524" layer="91"/>
 <junction x="48.26" y="38.1"/>
-<pinref part="U7" gate="G$1" pin="VIN"/>
-</segment>
-</net>
+</segment>
+</net>

Commit message: 100nF add to 3V3
Parts:
- added C4: 100n, rcl:C-EUC0603
Connections:
- net +3V3: now also C4.1
- net GND: now also C4.2
Changed lines of the file:
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@@
 <part name="C5" library="rcl" deviceset="C-EU" device="C0603" value="1u"/>
 <part name="GND12" library="supply1" library_urn="urn:adsk.eagle:library:371" deviceset="GNDIO" device=""/>
+<part name="C4" library="rcl" library_urn="urn:adsk.eagle:library:334" deviceset="C-EU" device="C0603" package3d_urn="urn:adsk.eagle:package:23616/2" value="100n"/>
+<part name="GND13" library="supply1" library_urn="urn:adsk.eagle:library:371" deviceset="GND" device=""/>
+<part name="P+6" library="supply1" library_urn="urn:adsk.eagle:library:371" deviceset="+3V3" device=""/>
 </parts>
 <sheets>
@@
 </instance>
 <instance part="GND12" gate="G$1" x="48.26" y="17.78" smashed="yes"/>
+<instance part="C4" gate="G$1" x="259.08" y="76.2" smashed="yes">
+<attribute name="NAME" x="260.604" y="76.581" size="1.778" layer="95"/>
+<attribute name="VALUE" x="260.604" y="71.501" size="1.778" layer="96"/>
+</instance>
+<instance part="GND13" gate="1" x="259.08" y="66.04" smashed="yes">
+<attribute name="VALUE" x="256.54" y="63.5" size="1.778" layer="96"/>
+</instance>
+<instance part="P+6" gate="G$1" x="259.08" y="86.36" smashed="yes">
+<attribute name="VALUE" x="259.08" y="86.36" size="1.778" layer="96" rot="R90"/>
+</instance>
 </instances>
 <busses>
@@
 <label x="48.26" y="17.78" size="1.778" layer="95" xref="yes"/>
 <pinref part="C5" gate="G$1" pin="2"/>
+</segment>
+<segment>
+<pinref part="C4" gate="G$1" pin="2"/>
+<pinref part="GND13" gate="1" pin="GND"/>
+<wire x1="259.08" y1="71.12" x2="259.08" y2="68.58" width="0.1524" layer="91"/>
 </segment>
 </net>
@@
 <wire x1="154.94" y1="78.74" x2="154.94" y2="86.36" width="0.1524" layer="91"/>
 </segment>
-</net>
+<segment>
+<pinref part="P+6" gate="G$1" pin="+3V3"/>
+<wire x1="259.08" y1="83.82" x2="259.08" y2="78.74" width="0.1524" layer="91"/>
+<pinref part="C4" gate="G$1" pin="1"/>
+</segment>
+</net>
