File: CRSpill.brd (EAGLE design)
At the start: 70 x 22.2 mm, 23 parts, among them IC1 7805DT, IC2 BLUE_PILL, IC3 NCV7351D1E, J3 MA04-1, SW1 SWITCH_TACTILETOP, U1 STM32F103C8, U7 XC6206, X1 8P8C-LED

Commit message: 水晶他諸々修正済み
Parts:
- moved C2 4.67 mm to (29.8, 11.4), turned to 180 degrees
- moved U$6 1.80 mm to (32.5, 8.96)
- moved C17 0.97 mm to (30.6, 14.8), turned to 0 degrees
Routing:
- net GND: track 156.2 -> 183.4 mm, vias 1 -> 0
- net +5V: track 86.2 -> 64.7 mm, vias 0 -> 1
- net CANTX: track 33.9 -> 25.0 mm, vias 1 -> 0
- net !RESET: track 72.5 -> 66.3 mm, vias 1 -> 3
- net N$11: track 8.72 -> 3.69 mm, vias 2 -> 0
- net SWDIO: track 32.3 -> 27.6 mm
- net !EMS: track 71.4 -> 74.4 mm
- net PA0: track 13.7 -> 11.2 mm, vias 2 -> 1
- net VBAT: track 22.7 -> 21.4 mm, vias 1 -> 0
- net N$19: track 2.65 -> 3.73 mm
- net +3V3: track 85.6 -> 86.6 mm, vias 4 -> 5
- net CANRX: track 37.4 -> 37.1 mm, vias 2 -> 1
- net PB7: vias 1 -> 0
Other:
- board text added: "CRSpill by ykc"

Commit message: boot0他
Parts:
- added BOOT0: (no value), jumper:SJ_2
Connections:
- net +3V3: now also BOOT0.1
- net BOOT0: now also BOOT0.2
- net GND: now also BOOT0.3
Routing:
- net GND: track 183.4 -> 176.8 mm
- net BOOT0: track 0.00 -> 6.59 mm, vias 0 -> 1
- net +3V3: track 86.6 -> 89.7 mm
- added copper zone on layer 1, net GND
- added copper zone on layer 16, net GND

Commit message: debug repair
Parts:
- moved C3 3.35 mm to (21.9, 10.7), turned to 90 degrees
- moved IC1 1.90 mm to (26.6, 11.5)
- moved C2 1.72 mm to (31.2, 12.4), turned to 270 degrees
- moved C17 1.00 mm to (31.6, 14.8)
- turned C1 to 90 degrees
Routing:
- net GND: track 176.8 -> 180.3 mm, vias 0 -> 2
- net PA0: track 11.2 -> 14.5 mm
- net +5V: track 64.7 -> 62.3 mm
- net CANTX: track 25.0 -> 26.4 mm
- net N$3: track 7.06 -> 8.14 mm

Commit message: 電解コンデンサ1個表面実装用に変更
Parts:
- removed C17: 22u, rcl:E2-5
- added C5: 1u, rcl:C0603
Connections:
- net +5V: now also C5.1; no longer C17.+
- net GND: now also C5.2; no longer C17.-
Routing:
- net +5V: track 62.3 -> 62.8 mm, vias 1 -> 2
- net GND: track 180.3 -> 180.5 mm, vias 2 -> 3
Other:
- board text added: "+3V3"
- board text added: "+5V"
- board text added: "A0"
- board text added: "A1"
- board text added: "A10"
- board text added: "A11"
- board text added: "A12"
- board text added: "A15"
- board text added: "A2"
- board text added: "A3"
- board text added: "A4"
- board text added: "A5"
- board text added: "A6"
- board text added: "A7"
- board text added: "A8"
- board text added: "A9"
- board text added: "B0"
- board text added: "B1"
- board text added: "B10"
- board text added: "B11"
- board text added: "B12"
- board text added: "B13"
- board text added: "B14"
- board text added: "B15"
- board text added: "B3"
- board text added: "B4"
- board text added: "B5"
- board text added: "B6"
- board text added: "B7"
- board text added: "B8"
- board text added: "B9"
- board text added: "C13"
- board text added: "C14"
- board text added: "C15"
- board text added: "EMS"
- board text added: "GND"
- board text added: "RESET"
- board text added: "VBAT"
Changed lines of the file:
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@@
 <drawing>
 <settings>
-<setting alwaysvectorfont="yes"/>
+<setting alwaysvectorfont="no"/>
 <setting verticaltext="up"/>
 </settings>
@@
 <wire x1="-0.5" y1="22.76" x2="-0.5" y2="0.6" width="0" layer="20"/>
 <text x="48" y="7" size="1.778" layer="21">CRSpill by ykc</text>
+<text x="16.1" y="21.2" size="0.6096" layer="21">+3V3</text>
+<text x="18.7" y="21.2" size="0.6096" layer="21">GND</text>
+<text x="64.5" y="1.4" size="0.6096" layer="21">GND</text>
+<text x="61.9" y="1.3" size="0.6096" layer="21">GND</text>
+<text x="59.3" y="1.3" size="0.6096" layer="21">+3V3</text>
+<text x="56.4" y="1.3" size="0.6096" layer="21">RESET</text>
+<text x="54.4" y="1.3" size="0.6096" layer="21">B11</text>
+<text x="51.8" y="1.4" size="0.6096" layer="21">B10</text>
+<text x="49.6" y="1.3" size="0.6096" layer="21">B1</text>
+<text x="47" y="1.3" size="0.6096" layer="21">B0</text>
+<text x="44.5" y="1.3" size="0.6096" layer="21">A7</text>
+<text x="42" y="1.3" size="0.6096" layer="21">A6</text>
+<text x="39.4" y="1.3" size="0.6096" layer="21">A5</text>
+<text x="36.8" y="1.3" size="0.6096" layer="21">A4</text>
+<text x="34.3" y="1.3" size="0.6096" layer="21">A3</text>
+<text x="31.8" y="1.3" size="0.6096" layer="21">A2</text>
+<text x="29.4" y="1.2" size="0.6096" layer="21">A1</text>
+<text x="26.8" y="1.3" size="0.6096" layer="21">A0</text>
+<text x="23.9" y="1.3" size="0.6096" layer="21">C15</text>
+<text x="21.4" y="1.3" size="0.6096" layer="21">C14</text>
+<text x="18.8" y="1.3" size="0.6096" layer="21">C13</text>
+<text x="16" y="1.3" size="0.6096" layer="21">VBAT</text>
+<text x="21.4" y="21.2" size="0.6096" layer="21">+5V</text>
+<text x="18.7" y="5.9" size="0.6096" layer="21">EMS</text>
+<text x="24.3" y="21.2" size="0.6096" layer="21">B9</text>
+<text x="26.7" y="21.2" size="0.6096" layer="21">B8</text>
+<text x="29.1" y="21.2" size="0.6096" layer="21">B7</text>
+<text x="31.8" y="21.2" size="0.6096" layer="21">B6</text>
+<text x="34.3" y="21.2" size="0.6096" layer="21">B5</text>
+<text x="36.9" y="21.2" size="0.6096" layer="21">B4</text>
+<text x="39.4" y="21.2" size="0.6096" layer="21">B3</text>
+<text x="41.8" y="21.1" size="0.6096" layer="21">A15</text>
+<text x="44.4" y="21.1" size="0.6096" layer="21">A12</text>
+<text x="46.9" y="21.1" size="0.6096" layer="21">A11</text>
+<text x="49.4" y="21.1" size="0.6096" layer="21">A10</text>
+<text x="52.2" y="21.1" size="0.6096" layer="21">A9</text>
+<text x="54.7" y="21.1" size="0.6096" layer="21">A8</text>
+<text x="57" y="21.1" size="0.6096" layer="21">B15</text>
+<text x="59.6" y="21.2" size="0.6096" layer="21">B14</text>
+<text x="62.1" y="21.2" size="0.6096" layer="21">B13</text>
+<text x="64.6" y="21.2" size="0.6096" layer="21">B12</text>
 </plain>
 <attributes>
@@
 <attribute name="VALUE" x="8.255" y="19.05" size="1.27" layer="27" rot="R270"/>
 </element>
-<element name="C17" library="rcl" package="E2-5" value="22u" x="31.56" y="14.8" smashed="yes">
-<attribute name="NAME" x="26.1" y="11.816" size="1.27" layer="25" ratio="10"/>
-<attribute name="VALUE" x="34.1" y="12.641" size="1.27" layer="27" ratio="10"/>
-</element>
 <element name="C16" library="rcl" package="C0603" value="100n" x="56.67" y="6.75" smashed="yes" rot="MR180">
 <attribute name="NAME" x="58.135" y="6.915" size="1.27" layer="26" rot="MR180"/>
@@
 <attribute name="POPULARITY" value="7" x="36.5" y="16.2" size="1.778" layer="28" rot="MR0" display="off"/>
 <attribute name="VALUE" x="36.6001" y="16.2" size="0.02" layer="28" rot="MR0"/>
+</element>
+<element name="C5" library="rcl" package="C0603" value="1u" x="31.6" y="15" smashed="yes" rot="MR180">
+<attribute name="NAME" x="30.965" y="14.365" size="1.27" layer="26" rot="MR180"/>
+<attribute name="VALUE" x="30.965" y="16.905" size="1.27" layer="28" rot="MR180"/>
 </element>
 </elements>
@@
 <contactref element="U1" pad="23"/>
 <contactref element="U1" pad="8"/>
-<contactref element="C17" pad="-"/>
 <contactref element="C16" pad="2"/>
 <contactref element="C18" pad="2"/>
@@
 <wire x1="5.1054" y1="9.8298" x2="5.08" y2="9.9" width="0.1524" layer="1"/>
 <wire x1="36.2712" y1="15.1638" x2="36.2712" y2="14.7828" width="0.1524" layer="1"/>
-<wire x1="35.8902" y1="15.5448" x2="36.2712" y2="15.1638" width="0.1524" layer="1"/>
-<wire x1="33.169315625" y1="15.5448" x2="35.8902" y2="15.5448" width="0.1524" layer="1"/>
+<wire x1="36.2712" y1="15.1638" x2="35.8902" y2="15.5448" width="0.1524" layer="1"/>
 <wire x1="36.2712" y1="14.7828" x2="36.305003125" y2="14.74113125" width="0.1524" layer="1"/>
-<wire x1="33.169315625" y1="15.5448" x2="32.576" y2="14.8" width="0.1524" layer="1"/>
 <wire x1="43.434" y1="8.6106" x2="43.434" y2="8.2296" width="0.1524" layer="1"/>
 <wire x1="42.3672" y1="9.6774" x2="42.4053" y2="9.6393" width="0.1524" layer="1"/>
@@
 <wire x1="20.574" y1="15.9" x2="20.574" y2="16.3068" width="0.1524" layer="1"/>
 <wire x1="19.6596" y1="19.05" x2="19.63" y2="19.09" width="0.1524" layer="1"/>
-<wire x1="32.576" y1="14.8" x2="32.576" y2="15.0678" width="0.1524" layer="1"/>
 <wire x1="32.576" y1="15.0678" x2="31.9466" y2="15.6972" width="0.1524" layer="1"/>
 <wire x1="20.574" y1="15.6972" x2="31.9466" y2="15.6972" width="0.1524" layer="1"/>
@@
 <wire x1="11.7348" y1="15.9258" x2="11.67" y2="15.93" width="0.1524" layer="16"/>
 <wire x1="15.3162" y1="10.2108" x2="14.79" y2="10.285" width="0.1524" layer="16"/>
-<wire x1="33.084240625" y1="13.4112" x2="47.0916" y2="13.4112" width="0.1524" layer="16"/>
+<wire x1="47.0916" y1="13.4112" x2="33.084240625" y2="13.4112" width="0.1524" layer="16"/>
 <wire x1="47.0916" y1="13.4112" x2="47.15" y2="13.42" width="0.1524" layer="16"/>
-<wire x1="33.084240625" y1="13.4112" x2="32.576" y2="14.8" width="0.1524" layer="16"/>
 <wire x1="32.54" y1="8.96" x2="31.96" y2="8.96" width="0.1524" layer="1"/>
 <wire x1="31.96" y1="8.96" x2="31" y2="8" width="0.1524" layer="1"/>
@@
 <via x="30" y="11.52" extent="1-16" drill="0.35"/>
 <wire x1="30" y1="11.52" x2="32.576" y2="14.096" width="0.5" layer="1"/>
-<wire x1="32.576" y1="14.096" x2="32.576" y2="14.8" width="0.5" layer="1"/>
 <wire x1="26.62" y1="9" x2="29" y2="11.38" width="0.5" layer="16"/>
 <wire x1="29" y1="11.38" x2="29" y2="11.52" width="0.5" layer="16"/>
+<contactref element="C5" pad="2"/>
+<wire x1="33.084240625" y1="13.4112" x2="32.45" y2="14.045440625" width="0.1524" layer="16"/>
+<wire x1="32.45" y1="14.045440625" x2="32.45" y2="15" width="0.1524" layer="16"/>
+<wire x1="33.053" y1="15.5448" x2="32.576" y2="15.0678" width="0.1524" layer="1"/>
+<wire x1="35.8902" y1="15.5448" x2="33.053" y2="15.5448" width="0.1524" layer="1"/>
+<via x="32.576" y="15.0678" extent="1-16" drill="0.35"/>
+<wire x1="32.576" y1="14.096" x2="32.576" y2="15.0678" width="0.5" layer="1"/>
 </signal>
 <signal name="N$2" class="1">
@@
 <contactref element="IC3" pad="5"/>
 <contactref element="IC2" pad="P$38"/>
-<contactref element="C17" pad="+"/>
 <contactref element="C16" pad="1"/>
 <contactref element="U7" pad="3"/>
@@
 <wire x1="27.9" y1="16.3" x2="26.0604" y2="17.181546875" width="0.5" layer="16"/>
 <wire x1="27.9" y1="16.3" x2="28.9" y2="16.3" width="0.5" layer="16"/>
-<wire x1="24.4792" y1="9.7726" x2="21.836" y2="9.7726" width="0.5" layer="1"/>
-<wire x1="29.5066" y1="14.8" x2="24.4792" y2="9.7726" width="0.5" layer="1"/>
 <wire x1="21.836" y1="9.7726" x2="21.836" y2="9.829375" width="0.5" layer="16"/>
 <wire x1="21.836" y1="9.829375" x2="21.85" y2="9.83" width="0.5" layer="16"/>
-<wire x1="29.5066" y1="14.8" x2="30.544" y2="14.8" width="0.5" layer="1"/>
 <via x="21.836" y="9.7726" extent="1-16" drill="0.35"/>
 <wire x1="19.49" y1="7.745" x2="20.745" y2="7.745" width="0.5" layer="16"/>
@@
 <wire x1="31.5722" y1="12.8778" x2="31.23" y2="13.22" width="0.5" layer="16"/>
 <wire x1="41.6052" y1="12.8778" x2="31.5722" y2="12.8778" width="0.5" layer="16"/>
-<wire x1="31.23" y1="13.22" x2="30.544" y2="13.906" width="0.5" layer="16"/>
-<wire x1="30.544" y1="13.906" x2="30.544" y2="14.8" width="0.5" layer="16"/>
-<wire x1="30.544" y1="14.8" x2="29.044" y2="16.3" width="0.5" layer="16"/>
-<wire x1="29.044" y1="16.3" x2="28.9" y2="16.3" width="0.5" layer="16"/>
+<contactref element="C5" pad="1"/>
+<wire x1="28.9" y1="16.3" x2="30.2" y2="15" width="0.5" layer="16"/>
+<wire x1="30.2" y1="15" x2="30.75" y2="15" width="0.5" layer="16"/>
+<via x="30.75" y="15" extent="1-16" drill="0.35"/>
+<wire x1="31.23" y1="13.22" x2="30.75" y2="13.7" width="0.5" layer="16"/>
+<wire x1="30.75" y1="13.7" x2="30.75" y2="15" width="0.5" layer="16"/>
+<wire x1="21.836" y1="9.7726" x2="25.5226" y2="9.7726" width="0.5" layer="1"/>
+<wire x1="25.5226" y1="9.7726" x2="30.75" y2="15" width="0.5" layer="1"/>
 </signal>
 <signal name="CANTX">

Commit message: 改造完了
Parts:
- moved C18 32.8 mm to (24.8, 13.8), flipped to the top
- moved U7 30.1 mm to (23.9, 10.7), flipped to the top
- moved C16 29.7 mm to (27.9, 14.1), flipped to the top
- moved C20 8.98 mm to (53.5, 7.95), flipped to the top, turned to 180 degrees
- moved R17 6.37 mm to (60.0, 8.97), flipped to the top, turned to 180 degrees
- moved R16 4.82 mm to (52.0, 10.1), flipped to the top, turned to 0 degrees
- moved BOOT0 4.00 mm to (32.5, 16.2)
- moved C5 3.86 mm to (27.9, 16.1), flipped to the top
- moved C2 3.38 mm to (27.9, 12.0), flipped to the top, turned to 180 degrees
- moved C3 2.73 mm to (19.4, 9.38), flipped to the top
- moved SW1 2.24 mm to (57.0, 13.2)
- moved C1 1.00 mm to (20.5, 14.6)
- moved F1 1.00 mm to (16.3, 13.7)
- moved IC3 1.00 mm to (17.1, 9.38)
- moved R1 1.00 mm to (14.6, 7.37)
Routing:
- net GND: track 180.5 -> 0.00 mm, vias 3 -> 62
- net !RESET: track 66.3 -> 31.8 mm, vias 3 -> 0
- net +5V: track 62.8 -> 35.2 mm, vias 2 -> 3
- net +3V3: track 89.7 -> 79.7 mm, vias 5 -> 6
- net SWCLK: track 37.2 -> 27.7 mm, vias 0 -> 1
- net CANRX: track 37.1 -> 27.8 mm, vias 1 -> 0
- net LED_CAN: track 36.3 -> 31.3 mm
- net CANTX: track 26.4 -> 30.5 mm
- net PB1: track 10.2 -> 13.8 mm, vias 0 -> 1
- net PA0: track 14.5 -> 11.1 mm, vias 1 -> 0
- net PB10: track 12.0 -> 15.0 mm, vias 0 -> 1
- net PB6: track 7.99 -> 10.1 mm, vias 0 -> 1
- net N$16: track 2.55 -> 4.33 mm, vias 1 -> 0
- net N$2: track 19.3 -> 20.9 mm
- net !EMS: track 74.4 -> 73.1 mm
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